File: KiCAD Files/podule_econet.kicad_sch (KiCad schematic)
At the start: 83 parts, among them IC1 68B54, IC10 SST39SF040, IC11 74HCT273, IC12 74HCT245, IC13 74HCT139, IC14 74HCT139, IC15 ATTINY45, IC2 74HCT132, IC3 74LS123, IC5 LM319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

Commit message: Updated for KiCAD V9
+ Updated 3D model file locations
Parts:
- added G1: LOGO, EconetPodule:AcornLogo2, symbol EconetPodule:AcornLogo2
- added LED1: Red, LED_THT:LED_D3.0mm, symbol Device:LED
- added LED2: Green, LED_THT:LED_D3.0mm, symbol Device:LED
- added LED3: Blue, LED_THT:LED_D3.0mm, symbol Device:LED
- added R32: 2K2, Resistor_THT:R_Axial_DIN0207_L6.3mm_D2.5mm_P10.16mm_Horizontal, symbol Device:R
- added R33: 330R, Resistor_THT:R_Axial_DIN0207_L6.3mm_D2.5mm_P10.16mm_Horizontal, symbol Device:R
- added R34: 20K, Resistor_THT:R_Axial_DIN0207_L6.3mm_D2.5mm_P10.16mm_Horizontal, symbol Device:R
Connections:
- net +5V: now also R32.1, R33.1, R34.1
- net Rx_Data: now reaches IC1.3 (Rx_Data), IC5.12, R4.2, R7.2
- net Rx_Data: now also LED2.1 (K)
- net Tx_Data: now reaches IC1.6 (Tx_Data), IC7.7 (Enable)
- net Tx_Data: now also LED1.1 (K)
- net Econet_Clk: now reaches IC1.27 (~{DCD}), IC3.12 (~{Q})
- net Econet_Clk: now also LED3.1 (K)
- new net: LED1.2 (A), R32.2
- new net: LED2.2 (A), R33.2
- new net: LED3.2 (A), R34.2
Other:
- note added: "Notes: Cathode / Short leg / Flat edge on inboard side of PCB Resistor values updated 23/02/25"
- moved on the sheet: C1, C10, C11, C12, C13, C14, C15, C16, C17, C18, C2, C3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
